File: Hardware/GWHMI/GWHMI.kicad_sch (KiCad schematic)
At the start: 20 parts, among them U1 DM-OLED096-636

Commit message: GWHMI: updated symbol fields SHIO88E: fixed silkscreen texts
Parts:
- R1: LCSC C17414 -> C17520; Order link 1 https://www.hestore.hu/prod_10040338.html -> https://www.hestore.hu/prod_10040677.html
- R2: LCSC C17414 -> C17661; Order link 1 https://www.hestore.hu/prod_10040338.html -> https://www.hestore.hu/prod_10027533.html
Changed lines of the file:
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@@
 			)
 		)
-		(property "Description" "10k, SMD 0805"
+		(property "Description" "2,2k, SMD 0805"
 			(at 80.01 88.9 0)
 			(effects
@@
 			)
 		)
-		(property "LCSC" "C17414"
+		(property "LCSC" "C17520"
 			(at 80.01 88.9 0)
 			(effects
@@
 			)
 		)
-		(property "Order link 1" "https://www.hestore.hu/prod_10040338.html"
+		(property "Order link 1" "https://www.hestore.hu/prod_10040677.html"
 			(at 80.01 88.9 0)
 			(effects
@@
 			)
 		)
-		(property "Description" "10k, SMD 0805"
+		(property "Description" "3k, SMD 0805"
 			(at 85.09 99.06 0)
 			(effects
@@
 			)
 		)
-		(property "LCSC" "C17414"
+		(property "LCSC" "C17661"
 			(at 85.09 99.06 0)
 			(effects
@@
 			)
 		)
-		(property "Order link 1" "https://www.hestore.hu/prod_10040338.html"
+		(property "Order link 1" "https://www.hestore.hu/prod_10027533.html"
 			(at 85.09 99.06 0)
 			(effects
